Commit message: Enhance circle tracking benchmark functionality and tests
- Added new parameters for velocity target integration and command actual error policy in test_config_loader.
- Updated test cases to validate new configuration options and added rejection tests for invalid configurations.
- Expanded rbsim_hardware_free_gate tests to include new snapshot fields related to command deadlines and send periods.
- Modified safety_policy tests to ensure serialization of new snapshot fields.
- Introduced a new script for comparing circle tracking benchmark results and generating markdown reports.
- Implemented unit tests for circle tracking benchmark helper functions to ensure correct behavior and threshold handling.
- Updated codex_gate.sh to include new benchmark runtime checks and configurations.
- Improved documentation and comments for clarity on new features and tests.

File: rb_servo_server/descriptions/urdf/rb3_730e.urdf (robot description, URDF)
Before this commit: robot rb3_730e, 10 links, 9 joints
Links:
- added link tool; visual mesh filename=../meshes/robots/rb3_730e/visual/tool/tool.STL scale=0.001 0.001 0.001
Joints:
- added joint tool_joint: type fixed, parent tcp, child tool, origin xyz=0.0 0.0 0.0 rpy=0.0 0.0 0.0
- joint tcp_joint: origin xyz=0.0 0.0 0.1 rpy=0.0 0.0 0.0 -> xyz=0.0 0.0 0.21616 rpy=0.0 0.0 0.0; parent link6 -> attachment_site

Commit message: Add unit tests for circle benchmark report, tracking benchmark, and circle ablation runner
- Implement tests for circle benchmark report helpers in `test_circle_benchmark_report.py` to validate comparison row handling, classification of baseline candidates, and report generation.
- Enhance `test_circle_tracking_benchmark.py` with tests for feedback controller help message, feedback formula correctness, and preflight rejection of real configurations.
- Introduce `test_run_circle_ablation.py` to validate matrix parsing, experiment validation, config overlay creation, and summary aggregation for circle ablation.
- Add a new STL file `tool.stl` for additional tooling support.

File: rb_servo_server/descriptions/urdf/rb3_730e.urdf (robot description, URDF)
Before this commit: robot rb3_730e, 11 links, 10 joints
Joints:
- joint tool_joint: parent tcp -> attachment_site

Commit message: feat: Enhance UmiDualCartesianConfig with new parameters and validation
- Added target_lpf_tau_sec, deadband_linear_m, deadband_angular_rad, linear_axis_signs, angular_axis_signs, and delta_frame to UmiDualCartesianConfig.
- Implemented validation checks for new parameters in UmiDualCartesianConfig.
- Updated _umi_dual_cartesian_config to handle new configuration fields.

feat: Integrate new UmiDualCartesianConfig parameters into action source

- Modified make_action_source to include target_lpf_tau_sec, deadband_linear_m, deadband_angular_rad, linear_axis_signs, angular_axis_signs, and delta_frame.

test: Add comprehensive tests for UmiDualCartesianActionSource behavior

- Implemented tests for axis signs mirroring, delta frame behavior, LPF smoothing, deadband functionality, and validation of new configuration parameters.
- Ensured that the new features are covered by unit tests to maintain code quality.

fix: Update physical_motion_expected handling in GUI models

- Changed _field_value to _field_value_non_null for physical_motion_expected to handle null values correctly.

test: Add tests for physical_motion_expected fallback behavior

- Created tests to verify that physical_motion_expected correctly falls back to cartesian_gate when null.

fix: Adjust URDF for accurate TCP positioning

- Updated the TCP joint origin in rb3_730e.urdf to reflect the correct fingertip plane position.

feat: Implement Spring-Mass-Damper pose tracking filter

- Added SmdPoseTracker and SmdPoseTrackerConfig for improved pose tracking in teleoperation.

fix: Improve IK seeding logic in CartesianController

- Updated IK seed logic to use the previously sent target instead of the actual state to prevent relay limit cycles.

test: Validate IK seeding behavior in unit tests

- Added tests to ensure that the IK controller uses the correct seed for joint targets.

File: rb_servo_server/descriptions/urdf/rb3_730e.urdf (robot description, URDF)
Before this commit: robot rb3_730e, 11 links, 10 joints
Joints:
- joint tcp_joint: origin xyz=0.0 0.0 0.21616 rpy=0.0 0.0 0.0 -> xyz=0.0 0.0 0.247642 rpy=0.0 0.0 0.0

Commit message: Add joint moving average and SMD pose tracker implementations
- Introduced JointMovingAverage class for computing moving averages of joint targets.
- Added SmdPoseTracker class for tracking pose with independent damping and frequency settings.
- Updated configuration validation to include moving average window and pose tracking parameters.
- Implemented tests for JointMovingAverage and SmdPoseTracker to ensure correct functionality.
- Created a Python script to bridge rb_servo_server joint streams to PlotJuggler for visualization.

PLAN B

File: rb_servo_server/descriptions/urdf/rb3_730e.urdf (robot description, URDF)
Before this commit: robot rb3_730e, 11 links, 10 joints
Joints:
- joint tcp_joint: origin xyz=0.0 0.0 0.247642 rpy=0.0 0.0 0.0 -> (none)

Commit message: feat: Add floor constraint functionality and related tests
- Implemented twistLocalToStand function for converting local twists to stand frame.
- Enhanced command server to handle SetSafetyFloorZ command with floor_z_m parameter.
- Updated state publisher to include floor constraint telemetry in JSON output.
- Added tests for floor constraint behavior, ensuring correct handling of downward velocity and lateral movement.
- Created configuration tests for floor constraint parsing and validation.
- Introduced new self-collision tests to verify stand capsule configurations against initial poses.
- Added a script to run the full teleoperation stack with configurable parameters.

File: rb_servo_server/descriptions/urdf/rb3_730e.urdf (robot description, URDF)
Before this commit: robot rb3_730e, 11 links, 10 joints
Joints:
- joint tcp_joint: origin (none) -> xyz=0.0 0.0 0.247642 rpy=0.0 0.0 0.0
