Commit message: Enhance box detection functionality and safety configurations
- Added tests for box detection command endpoint and debounce behavior in `test_gui_contracts.py`.
- Implemented box detection command client with control schema in `BoxDetectCommandClient`.
- Updated safety limits for J3 (elbow) in `stack_real.yaml` and `stack_sim.yaml` to reflect physical constraints.
- Adjusted URDF files to maintain accurate joint limits for elbow joint.
- Introduced a utility function to read joint limits from URDF files in `config.cpp`.
- Updated tests to validate new safety limits and configurations.
- Added a new script `analyze_collision_jerk.py` for analyzing jerk in servo logs to identify potential causes of jerky motion.

File: rb_servo_server/descriptions/urdf/rb3_730e.urdf (robot description, URDF)
Before this commit: robot rb3_730e, 11 links, 10 joints
Joints:
- joint elbow_joint: limit lower=-6.2832 upper=6.2832 effort=150.0 velocity=3.141592653589793 -> lower=-2.618 upper=2.618 effort=150.0 velocity=3.141592653589793

File: rb_servo_server/descriptions/urdf/rb3_730e_pika_articulated.urdf (robot description, URDF)
Before this commit: robot rb3_730e, 13 links, 12 joints
Joints:
- joint elbow_joint: limit lower=-6.2832 upper=6.2832 effort=150.0 velocity=3.141592653589793 -> lower=-2.618 upper=2.618 effort=150.0 velocity=3.141592653589793

Commit message: Remove unused data analysis and force control implementations; update VM stack script for host-only networking configuration.

File: rb_servo_server/descriptions/urdf/rb3_730e.urdf (robot description, URDF)
Before this commit: robot rb3_730e, 11 links, 10 joints
Links:
- added link ft_sensor_base
- added link ft_sensor_measurement
Joints:
- added joint ft_sensor_base_joint: type fixed, parent attachment_site, child ft_sensor_base, origin xyz=0.0 0.0 0.015 rpy=0.0 0.0 1.5707963267948966
- added joint ft_sensor_measurement_joint: type fixed, parent ft_sensor_base, child ft_sensor_measurement, origin xyz=0.0 0.0 0.030 rpy=0.0 0.0 0.0

File: rb_servo_server/descriptions/urdf/rb3_730e_pika_articulated.urdf (robot description, URDF)
Before this commit: robot rb3_730e, 13 links, 12 joints
Links:
- added link ft_sensor_base
- added link ft_sensor_measurement
Joints:
- added joint ft_sensor_base_joint: type fixed, parent attachment_site, child ft_sensor_base, origin xyz=0.0 0.0 0.015 rpy=0.0 0.0 1.5707963267948966
- added joint ft_sensor_measurement_joint: type fixed, parent ft_sensor_base, child ft_sensor_measurement, origin xyz=0.0 0.0 0.030 rpy=0.0 0.0 0.0
