Commit message: Use Pika gripper as default tool mesh in rb3_730e URDF
Swap the tool link's visual mesh from tool.STL to the Pika gripper
(pika_gripper.STL). The Pika mesh is authored mount-at-z0 / body-+Z, so
the original roll=pi flip is dropped (rpy 0,0,pi/2) to seat it on the
flange with fingers pointing along the tool approach axis. Both arms load
this URDF, so the Pika gripper is now the default on left and right.

Also add tools/view_gripper_posed.py: a standalone viser viewer that poses
both arms at the InitMotion joint angles (mock GUI has no servo state) so
the link6-mounted gripper can be inspected without the servo server.

Co-Authored-By: Claude Opus 4.8 (1M context) <noreply@anthropic.com>

File: rb_servo_server/descriptions/urdf/rb3_730e.urdf (robot description, URDF)
Before this commit: robot rb3_730e, 11 links, 10 joints
Links:
- link tool: geometry visual mesh filename=../meshes/robots/rb3_730e/visual/tool/pika_gripper.STL scale=0.001 0.001 0.001

Commit message: fix(servo): decouple per-arm IK failure, widen elbow IK limit, add joint-limit + self-collision diagnostics
Single-arm InitMotion during flow could freeze BOTH arms. Two root causes,
found via make-run logs + servo_log telemetry, fixed here:

1. Per-arm IK-failure coupling (dual_arm_servo_loop): the loop blanket-held
   BOTH arms on any non-Ok command verdict, discarding the per-arm hold that
   computeServoTarget already encodes. A left-arm flow IK failure thus froze a
   right-arm InitMotion (and vice-versa). Now applySafety runs on `desired`
   unconditionally so a healthy arm keeps moving while only the failed arm
   holds; the command verdict is still surfaced for telemetry. Generalizes to
   every dual-arm scenario (single chokepoint). New regression test.

2. Elbow IK joint limit: rb3_730e*.urdf capped elbow_joint at +/-150 deg while
   the rbpodo raw controller range is +/-360. A normal picking trajectory drove
   the elbow to 150 deg and IK failed (reason=joint_limit), freezing the arm.
   Widened both URDFs' elbow limit to +/-6.2832 rad (+/-360 deg).

Diagnostics added:
- IK joint_limit now names the pinned joint: IkResult/CartesianSolveTelemetry
  carry joint_limit_worst_{index,margin_deg}; throttled WARN in the solver; new
  CSV columns {left,right}_cart_ik_joint_limit_{index,margin_deg}.
- self_collision_{min_clearance_m,pair} CSV columns so a controller
  op_stat_self_collision (1005) latch can be cross-checked against the server's
  own mesh proximity.

rbpodo op_stat parsing fixed to spec (rb_cobot_docs item 33/35): the suspect
fallback read the RAW op_stat_collision_occur / op_stat_self_collision, which
include reserved/out-collision-source/time-zone bits, risking false positives.
Only the low bits are valid (already masked in the main checks), so the raw
fallback for both is removed; soft_estop (plain 0/1) is unchanged. Malformed
values still fail-closed via the generic diagnostics_suspect path. Tests updated.

Co-Authored-By: Claude Opus 4.8 (1M context) <noreply@anthropic.com>

File: rb_servo_server/descriptions/urdf/rb3_730e.urdf (robot description, URDF)
Before this commit: robot rb3_730e, 11 links, 10 joints
Joints:
- joint elbow_joint: limit lower=-2.618 upper=2.618 effort=150.0 velocity=3.141592653589793 -> lower=-6.2832 upper=6.2832 effort=150.0 velocity=3.141592653589793

File: rb_servo_server/descriptions/urdf/rb3_730e_pika_articulated.urdf (robot description, URDF)
Before this commit: robot rb3_730e, 13 links, 12 joints
Joints:
- joint elbow_joint: limit lower=-2.618 upper=2.618 effort=150.0 velocity=3.141592653589793 -> lower=-6.2832 upper=6.2832 effort=150.0 velocity=3.141592653589793

Commit message: Render the RB5 arms in rb_gui, at the accuracy the operator judges by
The stand was fixed last commit; the ARMS were still RB3-shaped, which is worse than
it sounds -- RB3's links are 286/344 mm against RB5's 425/392, so the render
disagreed with the robot by more than a link length while looking plausible.

_robot_urdf_path() now returns rb5_850e_pika_articulated.urdf, generated alongside
the other two so its arm chain cannot drift from the IK model (asserted: 0.000e+00
deviation across every shared frame). It is a separate file from rb5_850e.urdf on
purpose -- its two prismatic finger joints would change the DOF of the model the C++
FK/IK loads.

MESH CHOICE. The operator needs to read 1-2 mm clearances off this render, which
rules out the collision hulls (already vendored, 0 MB, but convexity inflates them
3.9-57.8% -- they would misstate the exact gap being judged). Between upstream's two
visual sets: they are the same object (extents agree to 0.0002 mm) at different
tessellation, 142k vs 739k triangles. Measured the coarser one's surface deviation
from the finer by sampling 30k points per link: p50 0.0000 mm, p99 <= 0.063 mm, max
0.271 mm. That is an order below the threshold that matters, for 26 MB instead of
69 MB, so the .dae set is vendored.

The pika meshes are now ONE set in one directory. The hulls had moved to rb5_850e
last commit while the raw meshes stayed behind, which split a single physical gripper
across two robot trees and forced tools/eval_live_pose.cpp to carry two prefixes.
Moving the rest and repointing all consumers removes the duplication and the split.

Also swept the remaining RB3 assumptions out of the GUI and the asset pipeline:
reach-envelope and IK-infeasible overlays now load the RB5 files (both regenerated
here), and status_panel stripped the literal "dual_rb3_730e_" from collision link
names, which silently stopped shortening them once the prefix became dual_rb5_850e_
-- it now strips whatever "dual_<model>_" the URDF uses. tools/reach_envelope.py and
tools/ik_infeasible_region.py had RB3 baked into their defaults and their printed
headings; both are robot-agnostic now.

Two test aborts on the way, both mine: the suite was run against a stale build after
the mesh move, and one path in test_init_motion_planner.cpp is split across a string
-literal concatenation so the repo-wide grep for it came up empty. Full runs after
fixing: ctest 43/43, rb_gui 308/308, generator --check MATCH on all three URDFs,
--check-config clean on both profiles. policy_runner still not runnable here (no
torch), unchanged and untouched.

Co-Authored-By: Claude Opus 5 <noreply@anthropic.com>

File: rb_servo_server/descriptions/urdf/rb3_730e.urdf (robot description, URDF)
Before this commit: robot rb3_730e, 13 links, 12 joints
Links:
- link tool: geometry visual mesh filename=../meshes/robots/rb5_850e/visual/tool/pika_gripper.STL scale=0.001 0.001 0.001

File: rb_servo_server/descriptions/urdf/rb3_730e_pika_articulated.urdf (robot description, URDF)
Before this commit: robot rb3_730e, 15 links, 14 joints
Links:
- link finger_left: geometry visual mesh filename=../meshes/robots/rb5_850e/visual/tool/pika_finger_left.STL scale=0.001 0.001 0.001
- link finger_right: geometry visual mesh filename=../meshes/robots/rb5_850e/visual/tool/pika_finger_right.STL scale=0.001 0.001 0.001
- link tool: geometry visual mesh filename=../meshes/robots/rb5_850e/visual/tool/pika_gripper_base.STL scale=0.001 0.001 0.001
