Commit message: Measure the RB5 pika tool offset instead of inheriting RB3's
tcp sat at attachment_site + 247.642 mm, carried over from RB3 because the gripper
and adapter did not change in the swap. The hardware disagrees: that number was
measured from RB3's attachment_site, and the two vendors do not put that frame on
the same physical plane. It is out by about 15 mm.

Two hand-parked contact poses, read with tools/rbpodo_read_state (both PARKED,
0.0000 deg sample spread):

  A  both TCPs touching the stand      tool axes [-0.77,-0.58,-0.27] [-0.87,0.37,-0.34]
  B  the two TCPs touching each other  tool axes [ 0.14,-0.98,-0.13] [-0.06,0.99,0.10]

At 247.642 mm, pose A left the tips 14.97 / 14.00 mm clear of a surface they were
touching, and pose B put the two tips 29.88 mm apart -- 14.94 mm per arm. Pose B is
the one that identifies the cause, because it never touches the stand and because
its tool axes are nearly orthogonal to pose A's: a mount position error cannot
produce the same along-the-tool-axis shortfall in both poses, while a tool-length
error does so by construction. So this also retires the hypothesis the first pose
suggested on its own -- that the stand or the mounts were ~15 mm off. They are not.
Left/right mount agreement remains 0.95 mm.

A combined fit over all three contact residuals gives 262.87 mm. With it the model
reproduces both contacts: pose B 29.88 -> 7.33 mm, pose A 14.97 -> 3.26 mm (left)
and 14.00 -> 0.37 mm (right). The few-mm residue is the precision of parking an arm
against a surface by hand, so the value is good to roughly +/-3 mm; the generator
records both poses so it can be re-derived if the gripper or adapter changes.

Only the single-arm model moves: the dual URDF's tcp is vestigial (the collision
monitor resolves attachment_site by name and never reads tcp), exactly as on RB3.

Co-Authored-By: Claude Opus 5 <noreply@anthropic.com>

File: rb_servo_server/descriptions/urdf/rb5_850e.urdf (robot description, URDF)
Before this commit: robot rb5_850e, 13 links, 12 joints
Joints:
- joint tcp_joint: origin xyz=0.0 0.0 0.247642 rpy=0.0 0.0 0.0 -> xyz=0.0 0.0 0.26287 rpy=0.0 0.0 0.0
