Commit message: Model the printed PLA+TPU tip, and stop trusting the CAD's finger pose
The factory pika finger was replaced on the hardware by the printed v15 tip: a
black PLA spine plus a #F3E600 95A TPU contact blade. rb_gui was still drawing
the factory one-piece finger, in one flat grey, from an undated mesh drop.

WHAT THE HARDWARE SAID, AND WHAT IT BROKE
Caliper across the two TPU tip faces at the open stop: ~98 mm, and the jaws
close to contact. None of the three CAD-pose predictions is that number (90.35
with the seating shift derived below, 94.33 without it, 94.04 for the factory
finger), because THE VENDOR CAD DOES NOT DRAW THE FINGERS AT THE OPEN STOP --
it draws them 3.8 mm/side inboard of it. The old finger travel inherited the
same unchecked premise: 0.047 was never measured, it was picked so that the CAD
pose would close to zero gap, so the two numbers appeared to confirm each other
while resting on the same assumption.

So the placement is anchored on the measurement. The meshes are baked at the
measured open stop, and the stroke follows from it (gap 0 at closed => 49.0 mm
per side). That also explains the "it closes to 0" observation cleanly: at
stroke 49 with a 98 mm open gap the tips meet exactly at 0 % with no preload.
The earlier prediction of a 3.69 mm overlap was an artefact of the 47 mm travel.

One gap measurement cannot split the CAD seating shift from the extra opening --
they only appear as (e - s) = 1.83 mm, so s=1.991/e=3.83 and s=0/e=1.83 both
give 98.0 exactly. Nothing here depends on the split, so BOLT_DATUM_SHIFT_MM is
kept only for the carriage datum check, which still passes: the placed finger's
seat plane and four M2 holes land on the carriage's own features (in
pika_gripper_base.STL, at URDF Z 145.30 and |X| 82.02/95.03) within 0.06 mm.

NEW GENERATOR
tools/make_pika_tool_meshes.py builds all 13 tool meshes from the v15 CAD, with
--check proving the committed files are its output (byte-identical, and stable
across rebuilds). The previous eight meshes were a copy with no recorded source
or transform, which is the asset that goes stale silently when the hardware
changes -- and did. Input digests are pinned so a swapped CAD fails loudly.

COLOURING
pika_gripper_base.STL is one mesh, so the tool rendered as a single grey. It is
now partitioned BY CONNECTED COMPONENT (a plane through Z 45 would slice the
sensor's cable connector, which spans Z 18..27 but belongs to the sensor) into
the two flange-side adapters, the RFT64 sensor, and the gripper; the split is an
exact partition of the original faces, asserted. Base mesh itself is untouched
and is still the collision/hull source, so the colouring is visual only.

DELIBERATELY UNCHANGED
PIKA_TIP_OFFSET_M / tcp_joint / tool_xyz_mm / applied_force_mm: carriage face ->
tip is 102.342 mm on the factory finger and 102.278 on v15, i.e. 0.064 mm in a
247.642 mm chain. Moving that would be noise dressed up as a measurement.

Still owed on hardware: tool_mass_kg / tool_com_mm are measured values (CM
`ft identify`) and the tip changed mass by tens of grams per side; and any grasp
width in millimetres was scaled through a 94.04 mm full-open model against a
real 98.0 mm full scale, a 4.2 % shift.

Verified: both generators --check clean (URDF 3/3, meshes 13/13); jaw maps
100 % -> 98.00 mm, 50 % -> 49.00, 0 % -> 0.00 with no interpenetration; rendered
colours read 183/76/43/33/#F3E600; rb_gui unittest failure set unchanged from
HEAD; compileall clean.

Co-Authored-By: Claude Opus 5 <noreply@anthropic.com>

File: rb_servo_server/descriptions/urdf/rb5_850e_pika_articulated.urdf (robot description, URDF)
Before this commit: robot rb5_850e, 15 links, 14 joints
Links:
- link finger_left: geometry visual mesh filename=../meshes/robots/rb5_850e/visual/tool/pika_finger_left_pla.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 scale=0.001 0.001 0.001; visual mesh filename=../meshes/robots/rb5_850e/visual/tool/pika_finger_left_tpu.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 scale=0.001 0.001 0.001
- link finger_right: geometry visual mesh filename=../meshes/robots/rb5_850e/visual/tool/pika_finger_right_pla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 scale=0.001 0.001 0.001; visual mesh filename=../meshes/robots/rb5_850e/visual/tool/pika_finger_right_tpu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 scale=0.001 0.001 0.001
- link tool: geometry visual mesh filename=../meshes/robots/rb5_850e/visual/tool/pika_gripper_body.STL scale=0.001 0.001 0.001; visual mesh filename=../meshes/robots/rb5_850e/visual/tool/pika_gripper_ft_senso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 scale=0.001 0.001 0.001
Joints:
- joint finger_left_joint: limit lower=0.0 upper=0.05 effort=20.0 velocity=0.5 -> lower=0.0 upper=0.049 effort=20.0 velocity=0.5
- joint finger_right_joint: limit lower=-0.05 upper=0.0 effort=20.0 velocity=0.5 -> lower=-0.049 upper=0.0 effort=20.0 velocity=0.5
