Commit message: Put attachment_site on the real tool mounting plane, 15.23 mm out
The previous commit corrected the measured attachment_site->tip distance to
262.87 mm by lengthening tcp. That put tcp in the right place for the wrong
reason, and left three other things wrong.

The gripper meshes say where the 15 mm belongs. pika_gripper_hull.STL spans
z [0, 247.642] mm: it is modelled from the gripper's own MOUNTING FACE, and its
tip plane is 247.642 mm out. The gripper is physically unchanged across the swap,
so mounting-face -> tip really is 247.642 mm, and the missing 15.23 mm therefore
sits between upstream's attachment_site and that face. attachment_site is simply
not on the tool mounting plane in the RB5 model, whereas it is in the RB3 one --
which is why the number did not transplant.

That distinction is not cosmetic, and every consequence of getting it wrong ran
the unsafe way:

  - collision_monitor.cpp attaches the pika hulls AT attachment_site with identity
    placement. An attachment_site 15 mm inboard makes the self-collision guard miss
    the outermost 15 mm of the real gripper -- the fingertips, i.e. the part that
    actually reaches things.
  - kinematics flange_link IS attachment_site, and the force path takes its pose to
    place F/T readings, so the moment arm was short by the same 15 mm.
  - ft_sensor_base / ft_sensor_measurement hang off it.

Moving the frame fixes tcp, the gripper hulls, the flange pose and the F/T chain
together, and needs no code change. tcp goes back to attachment_site + 247.642 mm,
the value with mesh provenance.

Verified after the move: link6 -> attachment_site 96.70 -> 111.93 mm;
attachment_site -> tcp 247.642 mm; attachment_site -> ft_sensor_measurement
45.000 mm, matching the 45 mm the force-control config documents. Both contact
poses still reproduce -- TCP-to-TCP 7.33 mm, stand 3.26 / 0.37 mm. Over 500 random
configurations every frame shared with upstream ver2 deviates by 0 except
attachment_site, which moves by exactly 15.230 mm.

The first attempt subtracted the shift and moved the frame INTO the wrist, doubling
both poses' residuals (TCP-to-TCP 59.87 mm); the component is negative, so outward
is away from zero. The sign is now covered by the contact re-verification above.

Co-Authored-By: Claude Opus 5 <noreply@anthropic.com>

File: rb_servo_server/descriptions/urdf/dual_rb5_850e_ver3.urdf (robot description, URDF)
Before this commit: robot dual_rb5_850e_ver2, 30 links, 29 joints
Joints:
- joint dual_rb5_850e_left_attachment_site_joint: origin xyz=0.0 -0.0967 0.0 rpy=1.57 0.0 0.0 -> xyz=0.000000 -0.111930 0.000000 rpy=1.57 0.0 0.0
- joint dual_rb5_850e_right_attachment_site_joint: origin xyz=0.0 -0.0967 0.0 rpy=1.57 0.0 0.0 -> xyz=0.000000 -0.111930 0.000000 rpy=1.57 0.0 0.0

File: rb_servo_server/descriptions/urdf/rb5_850e.urdf (robot description, URDF)
Before this commit: robot rb5_850e, 13 links, 12 joints
Joints:
- joint attachment_site_joint: origin xyz=0.0 -0.0967 0.0 rpy=1.57 0.0 0.0 -> xyz=0.000000 -0.111930 0.000000 rpy=1.57 0.0 0.0
- joint tcp_joint: origin xyz=0.0 0.0 0.26287 rpy=0.0 0.0 0.0 -> xyz=0.0 0.0 0.247642 rpy=0.0 0.0 0.0

Commit message: Fix the 90 deg stand misalignment in rb_gui by reading the URDF, not constants
Reported from hardware after the first RB5 `make run`: the stand renders rotated 90
deg away from the arms. rb_gui carried three values copied out of
dual_rb3_730e_ver5.urdf, and one of them is a robot-specific compensation:

    _DEFAULT_STAND_MESH_POSE = (0, 0, 0.001, 0, 0, -1.57078)

That is RB3's stand VISUAL origin verbatim, and its -90 deg exists only to undo
RB3's own base->stand joint of +90 deg. RB5's base->stand is identity and so is its
stand visual origin, so the compensation survived as a pure 90 deg error. The
collision-overlay frame had the same constant baked in as -math.pi/2.

Both are now derived:
  - _stand_visual_from_urdf() reads the stand link's mesh and origin.
  - _urdf_stand_to_world_pose() composes the fixed-joint chain from `stand` to the
    root and inverts it, which is what the overlay frame actually needs.
Checked against both robots: the derivation reproduces the old constant EXACTLY for
dual_rb3_730e_ver5 (-90.00 deg) and gives 0.00 deg for RB5 -- i.e. it was right for
the robot it was written for, and the swap is now a no-op here.

To make that possible the generator re-adds ONE visual to dual_rb5_850e_ver3.urdf,
the stand's, pointing at the stand mesh now vendored in this repo (1.6 MB). Arm
visuals stay dropped -- upstream's are 67 MB. The collision model is untouched: 49
geometries before and after, 0 missing, --check still MATCHes.

_DEFAULT_LEFT_POSE/_DEFAULT_RIGHT_POSE also moved to the RB5 mounts. Those matter
less (they are startup fallbacks; the live mounts arrive in the state manifest) but
they were visibly wrong for the first frames, and note the arms mirror in Y now.

Two tests pinned the RB3 behaviour as magic numbers and would have gone stale again
at the next swap, so they now assert the invariant instead: the GUI's mount fallbacks
must equal the tracked URDF's stand_<side>_arm_base origins, and the overlay frame
must equal the inverse of that URDF's world->stand. Verified the first genuinely
fails when pointed at the RB3 URDF via RB_GUI_UNIFIED_URDF. rb_gui 308/308.

STILL RB3 and NOT fixed here: _robot_urdf_path() returns rb3_730e_pika_articulated
.urdf, so the rendered ARMS are still RB3-shaped. Fixing it needs a display asset
decision (upstream RB5 visuals are 67 MB of .obj / 26 MB of .dae, against the 1.3 MB
of collision hulls already vendored), which is the operator's call.

Co-Authored-By: Claude Opus 5 <noreply@anthropic.com>

File: rb_servo_server/descriptions/urdf/dual_rb5_850e_ver3.urdf (robot description, URDF)
Before this commit: robot dual_rb5_850e_ver2, 30 links, 29 joints
Links:
- link stand: geometry visual mesh filename=../meshes/stands/dual_rb5_850e/dual_rb5_850e_stand_ver2.stl scale=0.001 0.001 0.001

Commit message: Put attachment_site back on the flange, and rotate the ROI into the RB5 stand frame
Two things the first RB5 `make run` showed, both mine.

THE GRIPPER FLOATED OFF THE FLANGE. 1c81c93 moved attachment_site 15.23 mm out,
reasoning that the gripper meshes are modelled from their mounting face so the
missing distance had to sit between attachment_site and that face. The render says
otherwise, and so does the geometry: link6's visual mesh ends 96.57 mm from its
origin and upstream puts attachment_site at 96.70 mm, i.e. ON the flange face -- and
RB3 uses the SAME convention, its link6 ending at exactly 100.00 mm where its
attachment_site sits. My "the two vendors disagree" premise was simply wrong.

Both robots therefore measure the tool from the flange and should agree for the same
gripper. RB3 said 247.642 mm, the z-max of pika_gripper.STL; the hardware says
262.87 mm. Same convention, same adapter, same CAD, so what remains is that the
PHYSICAL tip is ~15 mm past that CAD -- consistent with the finger redesign this
gripper has been through (PLA spine + TPU blade, v7 -> v9), which the STL predates.
So attachment_site goes back to upstream's value and tcp carries the measured
262.87 mm. The flange-to-gripper gap is now 0.13 mm, both contact poses still
reproduce unchanged (TCP-to-TCP 7.33 mm, stand 3.26 / 0.37 mm), and ver3 is once
again kinematically identical to upstream at every frame (0.000e+00 over 400 configs)
rather than "identical except attachment_site".

Carried forward and NOT fixed, because it needs the current finger CAD rather than a
guess: the finger collision hulls are that same old geometry and stop at 247.642 mm,
so the self-collision guard misses the outermost ~15 mm of the real fingertips.

THE ROI BOX WAS 90 DEG OFF THE ARMS. roi_box bounds are STAND-FRAME, and the stand
frame convention changed with the robot: base->stand is +90 deg about Z on
dual_rb3_730e_ver5 and identity on dual_rb5_850e_ver3. The numbers were authored for
the old frame, so the same physical box now sat rotated -- and this one is enforced,
not merely drawn. Confirmed against hardware rather than by inspection: all four TCPs
from the two parked poses fall OUTSIDE the current box, including the pose with both
arms out over the table. Rotating by Rz(+90) puts the working pose inside and leaves
the pose touching the stand column outside, which is the correct answer for both.
The 2026-08-2x y_max tightening survives the rotation as the +0.300 x_min face.

Both profiles rotated. This assumes the table sits the same way relative to the
stand; the stand model itself changed (arm spacing +/-0.157 -> +/-0.197 m, height
0.580 -> 0.570), so the far faces are worth re-confirming against the real table
before they are leaned on.

ctest 43/43, rb_gui 308/308, generator --check MATCH, --check-config clean on both.

Co-Authored-By: Claude Opus 5 <noreply@anthropic.com>

File: rb_servo_server/descriptions/urdf/dual_rb5_850e_ver3.urdf (robot description, URDF)
Before this commit: robot dual_rb5_850e_ver2, 30 links, 29 joints
Joints:
- joint dual_rb5_850e_left_attachment_site_joint: origin xyz=0.000000 -0.111930 0.000000 rpy=1.57 0.0 0.0 -> xyz=0.0 -0.0967 0.0 rpy=1.57 0.0 0.0
- joint dual_rb5_850e_right_attachment_site_joint: origin xyz=0.000000 -0.111930 0.000000 rpy=1.57 0.0 0.0 -> xyz=0.0 -0.0967 0.0 rpy=1.57 0.0 0.0

File: rb_servo_server/descriptions/urdf/rb5_850e.urdf (robot description, URDF)
Before this commit: robot rb5_850e, 13 links, 12 joints
Joints:
- joint attachment_site_joint: origin xyz=0.000000 -0.111930 0.000000 rpy=1.57 0.0 0.0 -> xyz=0.0 -0.0967 0.0 rpy=1.57 0.0 0.0
- joint tcp_joint: origin xyz=0.0 0.0 0.247642 rpy=0.0 0.0 0.0 -> xyz=0.0 0.0 0.26287 rpy=0.0 0.0 0.0

File: rb_servo_server/descriptions/urdf/rb5_850e_pika_articulated.urdf (robot description, URDF)
Before this commit: robot rb5_850e, 15 links, 14 joints
Joints:
- joint attachment_site_joint: origin xyz=0.000000 -0.111930 0.000000 rpy=1.57 0.0 0.0 -> xyz=0.0 -0.0967 0.0 rpy=1.57 0.0 0.0
- joint tcp_joint: origin xyz=0.0 0.0 0.247642 rpy=0.0 0.0 0.0 -> xyz=0.0 0.0 0.26287 rpy=0.0 0.0 0.0

Commit message: Stand the pika gripper off the flange by its F/T adapter, exactly 15.000 mm
The gripper collision hulls were attached at attachment_site, i.e. bolted flat to the
flange. They are not: an F/T adapter stands the gripper off, so the whole gripper sat
15 mm nearer the wrist than it is. That runs BOTH ways wrong -- the guard missed the
outermost 15 mm of the fingertips, which is the part that reaches things, and covered
15 mm of empty air behind them.

THE NUMBER IS DERIVED, NOT FITTED. Both terms have provenance:

  flange -> gripper CAD origin = 45.0 - 30.0    = 15.000 mm
      45.0 mm is offset.xyz in the controller-manager RFT64-6A01-A preset (flange ->
      sensing reference origin); 30.0 mm is its sensor body. That preset's own comment
      says "adapter 13mm + sensor 30mm = 43mm", disagreeing with its VALUE by 2 mm.
  gripper CAD origin -> tip    = 247.642 mm     (pika_gripper.STL z-max)
  flange -> tip                = 262.642 mm

Against the hardware measurement of 262.870 mm (combined fit over three contact
residuals from two parked poses) that agrees to 0.228 mm -- and it also settles the
preset's internal disagreement, since the 13 mm reading would give 260.642 mm and miss
the measurement by 2.23 mm, outside its ~2 mm spread. The earlier guess that the
physical fingers were longer than their CAD is retracted: the operator confirms they
are the CAD fingers.

COVERAGE IS NOW CONTINUOUS, checked rather than assumed:
  adapter cylinder   flange -> 15.0 mm
  gripper base hull      15.0 -> 160.3 mm
  finger hulls          150.5 -> 262.6 mm
  tcp                            262.642 mm
No gap and no double cover. The adapter had been modelled by nothing at all: link6's
hull stops at the flange and the gripper hulls started at the gripper origin.

NO FALSE POSITIVES BY CONSTRUCTION. The adapter cylinder's 35 mm radius is the gripper
base's own mounting-face radius, which bounds it from above, and it sits entirely
inside link6's 82 x 87 mm silhouette -- so it cannot raise a proximity that link6 does
not already raise.

Mechanism: a gripper_attach_frame config key, defaulting to "attachment_site" so any
model without the new frame is untouched, pointed at the gripper_mount frame the RB5
URDFs now carry. A frame name rather than a magic offset, so the geometry lives in the
generated URDF where it is visible. Missing frames fail closed with the config key
named.

Tested: a new runGripperAttachFrame pins the default, asserts an unknown attach frame
throws rather than falling back, and measures the shift the monitor actually applies --
reports 15 mm. ctest 43/43, rb_gui 308/308, generator --check MATCH, --check-config
clean on both profiles.

Co-Authored-By: Claude Opus 5 <noreply@anthropic.com>

File: rb_servo_server/descriptions/urdf/dual_rb5_850e_ver3.urdf (robot description, URDF)
Before this commit: robot dual_rb5_850e_ver2, 30 links, 29 joints
Links:
- added link dual_rb5_850e_left_gripper_mount
- added link dual_rb5_850e_left_tool_adapter; collision cylinder length=0.015 radius=0.035
- added link dual_rb5_850e_right_gripper_mount
- added link dual_rb5_850e_right_tool_adapter; collision cylinder length=0.015 radius=0.035
Joints:
- added joint dual_rb5_850e_left_gripper_mount_joint: type fixed, parent dual_rb5_850e_left_attachment_site, child dual_rb5_850e_left_gripper_mount, origin xyz=0.0 0.0 0.015 rpy=0.0 0.0 0.0
- added joint dual_rb5_850e_left_tool_adapter_joint: type fixed, parent dual_rb5_850e_left_attachment_site, child dual_rb5_850e_left_tool_adapter, origin xyz=0.0 0.0 0.0 rpy=0.0 0.0 0.0
- added joint dual_rb5_850e_right_gripper_mount_joint: type fixed, parent dual_rb5_850e_right_attachment_site, child dual_rb5_850e_right_gripper_mount, origin xyz=0.0 0.0 0.015 rpy=0.0 0.0 0.0
- added joint dual_rb5_850e_right_tool_adapter_joint: type fixed, parent dual_rb5_850e_right_attachment_site, child dual_rb5_850e_right_tool_adapter, origin xyz=0.0 0.0 0.0 rpy=0.0 0.0 0.0

File: rb_servo_server/descriptions/urdf/rb5_850e.urdf (robot description, URDF)
Before this commit: robot rb5_850e, 13 links, 12 joints
Links:
- added link gripper_mount
- added link tool_adapter; collision cylinder length=0.015 radius=0.035
Joints:
- added joint gripper_mount_joint: type fixed, parent attachment_site, child gripper_mount, origin xyz=0.0 0.0 0.015 rpy=0.0 0.0 0.0
- added joint tool_adapter_joint: type fixed, parent attachment_site, child tool_adapter, origin xyz=0.0 0.0 0.0 rpy=0.0 0.0 0.0
- joint tcp_joint: origin xyz=0.0 0.0 0.26287 rpy=0.0 0.0 0.0 -> xyz=0.0 0.0 0.262642 rpy=0.0 0.0 0.0
- joint tool_joint: parent attachment_site -> gripper_mount

File: rb_servo_server/descriptions/urdf/rb5_850e_pika_articulated.urdf (robot description, URDF)
Before this commit: robot rb5_850e, 15 links, 14 joints
Links:
- added link gripper_mount
- added link tool_adapter; collision cylinder length=0.015 radius=0.035
Joints:
- added joint gripper_mount_joint: type fixed, parent attachment_site, child gripper_mount, origin xyz=0.0 0.0 0.015 rpy=0.0 0.0 0.0
- added joint tool_adapter_joint: type fixed, parent attachment_site, child tool_adapter, origin xyz=0.0 0.0 0.0 rpy=0.0 0.0 0.0
- joint finger_left_joint: parent attachment_site -> gripper_mount
- joint finger_right_joint: parent attachment_site -> gripper_mount
- joint tcp_joint: origin xyz=0.0 0.0 0.26287 rpy=0.0 0.0 0.0 -> xyz=0.0 0.0 0.262642 rpy=0.0 0.0 0.0
- joint tool_joint: parent attachment_site -> gripper_mount

Commit message: Revert the 15 mm tool standoff: the F/T sensor is inside pika_gripper.STL
a1aaaf8 moved the gripper collision geometry 15 mm off the flange and pushed tcp to
262.642 mm, on the strength of a contact measurement. Sectioning the CAD shows that was
wrong, and the number goes back to 247.642 mm.

WHAT THE SECTIONS SHOW (docs/reference/pika_gripper_sections.png, regenerated by
tools/plot_pika_gripper_sections.py). pika_gripper.STL's z = 1..55 mm is a Ø64 body
inside a Ø70 base sitting on a BOLT CIRCLE -- the RFT64-6A01-A sensor, not gripper
structure -- and the radius bulges to 60 mm at z = 20..25, which is the sensor's cable
connector, called out as "protruding past the body dia" in the controller-manager part
file. The stack ends near z = 45, exactly the sensor_offset_mm the force config
carries. So the STL starts AT THE FLANGE with the sensor inside it, and flange -> tip
is 247.642 mm. The force-control config agrees by the other route -- its tool_xyz_mm is
measured from the SENSOR, so 45 + 202.642 -- and was never in contradiction.

WHY THE MEASUREMENT MISLED. Two hand-parked poses each read ~15 mm long and their
agreement was taken as confirmation. It was not. The argument was that their tool axes
were "nearly orthogonal" so a common-mode error could not survive both; they are
60-67 deg apart. And nothing verified the premise the method rests on -- that the
FINGERTIP PLANE was what touched. Anything else on the gripper contacting first biases
the fit long, identically in both poses. A contact fit measures the distance to
whatever touched; it cannot say what that was. The CAD could answer this with no robot
at all and should have been asked first. That is written down in
docs/reference/pika_tool_geometry.md so the next person does not repeat it.

REVERTED: tcp 262.642 -> 247.642; the tool_adapter cylinder and gripper_mount frame are
gone from all three URDFs; the gripper_attach_frame config key, its plumbing through
config.cpp / dual_arm_servo_loop / CollisionMonitor, and the gripperGeometryOrigin
accessor are removed. Collision geometry is back to 49 in the unified URDF, and ver3 is
once again identical to upstream ver2 at every frame over 400 configurations
(0.000e+00). Tool chain verified: attachment_site 96.700 mm from link6 (flange face
96.57), ft_sensor_base +15.0, ft_sensor_measurement +45.0, tcp +247.642.

KEPT, because it is independently right: requireModelFrame / requireModelJoint still
fail closed on a prefix or frame the URDF does not carry. The test that exercised the
attach frame is replaced by one that pins exactly that -- a mismatched prefix must
throw, not degrade -- and it does.

Fallout fixed: test_safety_policy built its monitor from the sibling checkout's
dual_rb3_730e_ver5, so it broke when the left/right_prefix defaults moved to the RB5;
it now uses the tracked RB5 model with matching prefixes. Geometry counts 57/53 -> 55/51.

ctest 43/43, rb_gui 308/308, generator --check MATCH, --check-config clean on both.

Co-Authored-By: Claude Opus 5 <noreply@anthropic.com>

File: rb_servo_server/descriptions/urdf/dual_rb5_850e_ver3.urdf (robot description, URDF)
Before this commit: robot dual_rb5_850e_ver2, 34 links, 33 joints
Links:
- removed link dual_rb5_850e_left_gripper_mount
- removed link dual_rb5_850e_left_tool_adapter
- removed link dual_rb5_850e_right_gripper_mount
- removed link dual_rb5_850e_right_tool_adapter
Joints:
- removed joint dual_rb5_850e_left_gripper_mount_joint
- removed joint dual_rb5_850e_left_tool_adapter_joint
- removed joint dual_rb5_850e_right_gripper_mount_joint
- removed joint dual_rb5_850e_right_tool_adapter_joint

File: rb_servo_server/descriptions/urdf/rb5_850e.urdf (robot description, URDF)
Before this commit: robot rb5_850e, 15 links, 14 joints
Links:
- removed link gripper_mount
- removed link tool_adapter
Joints:
- removed joint gripper_mount_joint
- removed joint tool_adapter_joint
- joint tcp_joint: origin xyz=0.0 0.0 0.262642 rpy=0.0 0.0 0.0 -> xyz=0.0 0.0 0.247642 rpy=0.0 0.0 0.0
- joint tool_joint: parent gripper_mount -> attachment_site

File: rb_servo_server/descriptions/urdf/rb5_850e_pika_articulated.urdf (robot description, URDF)
Before this commit: robot rb5_850e, 17 links, 16 joints
Links:
- removed link gripper_mount
- removed link tool_adapter
Joints:
- removed joint gripper_mount_joint
- removed joint tool_adapter_joint
- joint finger_left_joint: parent gripper_mount -> attachment_site
- joint finger_right_joint: parent gripper_mount -> attachment_site
- joint tcp_joint: origin xyz=0.0 0.0 0.262642 rpy=0.0 0.0 0.0 -> xyz=0.0 0.0 0.247642 rpy=0.0 0.0 0.0
- joint tool_joint: parent gripper_mount -> attachment_site
