Commit message: stand: derive the collision model from upstream ver1, the stand this cell has
Upstream mo_robot_descriptions ships two RB5 stands and they are not
interchangeable: ver2 mounts each arm 15.00 mm further out along the 45 deg
plate -- (0.17036, +/-0.19707, 0.57036) vs (0.16285534, +/-0.18646447,
0.56285534), same rpy -- which puts the two arms 21.2 mm further apart in Y.
This repo has derived from ver2 since 2026-09-02 (de96559). It is the wrong one.

Measured three ways:

  * TAPE, no robot. The stand's full Y width is 507.3 mm under ver1 and 521.4
    under ver2. The operator measured ver1.
  * CONTACT FAR FROM THE MOUNT. Both arms hand-parked touching the stand,
    joints read off the boxes with rbpodo_read_state. The right arm reached
    down to the base column (z 0.11-0.21 m), far enough for the 15 mm to show:
    its contact point sits 7.00 mm off the true stand surface under ver2 and
    0.50 mm under ver1. The left arm touched just under its own mount, where
    arm and stand move together, and cannot tell the two apart (0.27 vs
    0.29 mm) -- that degeneracy is why this survived four days.
  * ARM TO ARM. A hand-built tip-to-wrist fixture reads 43.9 mm under ver2 and
    22.9 mm under ver1 against a physical ~15.

base_pose_in_stand MOVES WITH IT, NOT JUST THE URDF. The servo loop's FK/IK
takes the mounts from the stack config while the CollisionMonitor takes them
from the unified URDF, so fixing only one would have left the two models
disagreeing by 15 mm per arm. rb_gui asserts they match
(test_default_mounts_match_the_tracked_unified_urdf), and that assert is what
caught it here.

THE STAND COLLISION IS NOW HULLS ONLY. ver1 ships its stand as a raw 38k
triangle non-convex mesh and has none of ver2's primitive boxes, so the
generator drops that mesh -- coal keeps a non-convex mesh as a BVH, far
outside the per-eval budget the monitor's contract assumes -- and replaces it
with 20 CoACD hulls regenerated from ver1 using collision_ver2's exact
parameters. Measured on 6k surface samples with a half-space containment test:
100.0% coverage with no gap, over-approximating the true surface by mean 1.41
/ p95 8.76 / max 29.87 mm, against 4.59 / 14.76 / 37.80 for the ver2 set it
replaces. The guard therefore also got ~3x tighter where it brakes.

Verified: generator --check MATCH on all three URDFs, --check-config OK on
both stacks, ctest 47/47, 0 non-convex meshes kept as BVH, and the three
measured poses re-evaluated -- right-arm stand contact 7.00 -> -1.2..+2.6 mm,
tip-to-own-base closed loop unchanged at -4.9..+2.9 mm (the arm chains were
never the problem), fixture 43.9 -> 22.9 mm.

NOT FIXED HERE: a later contact pose (right gripper tips on the left wrist)
still reads 6.5 mm where the arms physically touch, so ~6.5 mm of arm-to-arm
error remains and still wants a relative mount calibration. It was 23.9 mm at
that pose under ver2.

Co-Authored-By: Claude Fable 5 <noreply@anthropic.com>

File: rb_servo_server/descriptions/urdf/dual_rb5_850e_ver3.urdf (robot description, URDF)
Before this commit: robot dual_rb5_850e_ver2, 33 links, 32 joints
Links:
- removed link base
- removed link base_site
- removed link stand_base_col
- removed link stand_body_shoulder
- removed link stand_body_upper
- link stand: geometry visual mesh filename=../meshes/stands/dual_rb5_850e/dual_rb5_850e_stand_ver1.stl scale=0.001 0.001 0.001
- link stand_collision: geometry collision mesh filename=../meshes/stands/dual_rb5_850e/collision_ver1/stand_hull_00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 scale=0.001 0.001 0.001; collision mesh filename=../meshes/stands/dual_rb5_850e/collision_ver1/stand_hull_00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 scale=0.001 0.001 0.001
Joints:
- removed joint base_fixed
- removed joint base_site_joint
- removed joint stand_base_col_fixed
- removed joint stand_body_shoulder_fixed
- removed joint stand_body_upper_fixed
- joint stand_fixed: parent base -> world
- joint stand_left_arm_base_fixed: origin xyz=0.17036 0.19707 0.57036 rpy=2.185913927779314 0.5231323161197823 -2.186648937497128 -> xyz=0.16285534 0.18646447 0.56285534 rpy=2.185913927779314 0.5231323161197823 -2.186648937497128; parent stand -> world
- joint stand_right_arm_base_fixed: origin xyz=0.17036 -0.19707 0.57036 rpy=2.1859138555489475 -0.5231322390070723 -0.9549437348744108 -> xyz=0.16285534 -0.18646447 0.56285534 rpy=2.1859138555489475 -0.5231322390070723 -0.9549437348744108; parent stand -> world

Commit message: mounts: apply the measured site calibration, fitted from 27 contact poses
The two arm mounts came from upstream's stand model. This replaces them with what
this cell actually measures, from contacts made on the robot itself.

METHOD. 27 hand-parked CONTACT poses, both jaws at the mechanical open stop: a tip
touching the other arm (6) or touching the stand (21, both arms). A contact means
the true clearance is 0, so the model's residual distance at that pose is pure model
error along that contact's normal -- one scalar equation each, which is why the
campaign chased normal DIVERSITY rather than pose count. Least squares for both
mounts, fitted through CollisionMonitor itself, so the model being fitted is the one
that gets enforced.

Three things had to be handled or the answer came out wrong:
  * The stand side is measured against the SOURCE STL, never the CoACD hulls --
    those over-approximate by mean 1.4 / max 29.9 mm.
  * The finger side uses the REAL printed mesh, not its convex hull: the hull fills
    the TPU blade's honeycomb (p50 0.04 mm, but p90 5.2 / max 15.2 mm). The gripper
    BASE hull is worse still, max 45.5 mm, and is not usable as a contact target.
  * A 7th unknown, a uniform stand SURFACE offset, is fitted alongside the mounts and
    then discarded. It comes out +1.94 +/- 0.32 mm -- the real stand sits that far
    outside its own STL. Omitting it from the FIT biased both mounts, because every
    stand contact carries it (arm<->stand residuals sat at -1.35 / -1.51 mm); omitting
    it from the MODEL is right, because it makes the guard conservative, not
    optimistic. With it: residual RMS 1.06 mm, leave-one-out 1.51 mm (from 2.39),
    condition number 3.2, against a 0.2-0.6 mm repeatability floor measured by
    touching one spot from different arm postures.

RESULT, and what it buys. left (-1.09, -1.89, -0.15), right (-1.87, +1.30, -0.71) mm.
Re-evaluating all 27 contacts through the corrected model (excluding 4 where the
closest pair switched, so before/after is not the same quantity): arm-to-arm error
2.54 -> 1.14 mm mean, and centred on zero (+1.74 -> +0.06). Arm-to-stand is unchanged
(spread 1.54 -> 1.64 mm). So this buys the CROSS-ARM pairs -- 187 arm<->arm plus the
9 gripper<->gripper pairs a handover runs through -- and nothing else, which is what
the statistics said all along: the relative term was the well-determined one, and it
converged 9.60 -> 6.59 -> 5.74 -> 4.54 -> 4.06 -> 3.33 mm as poses came in.

NOT RESOLVED: per-component sigma is 0.5-0.7 mm, so x and y are 2-3 sigma but BOTH z
terms are inside their own error bar (-0.15 +/- 0.7, -0.71 +/- 0.7). They are applied
because the least-squares estimate is unbiased, not because z is measured.

It lives in the generator as MOUNT_CALIBRATION_M so the URDF the guard loads and the
base_pose_in_stand the servo loop's FK/IK reads cannot drift apart; rb_gui asserts
they are equal. It is the one entry in that file that is a property of this cell
rather than of the robot, and it must be re-measured if an arm is ever unbolted.

Verified: generator --check MATCH on all three URDFs, --check-config OK on both
stacks, ctest 46/47 (preview_contact_qp fails identically with these changes stashed
-- a QP solver non-convergence unrelated to mounts).

Co-Authored-By: Claude Fable 5 <noreply@anthropic.com>

File: rb_servo_server/descriptions/urdf/dual_rb5_850e_ver3.urdf (robot description, URDF)
Before this commit: robot dual_rb5_850e_ver1, 28 links, 27 joints
Joints:
- joint stand_left_arm_base_fixed: origin xyz=0.16285534 0.18646447 0.56285534 rpy=2.185913927779314 0.5231323161197823 -2.186648937497128 -> xyz=0.16176534 0.18457447 0.56270534 rpy=2.185913927779314 0.5231323161197823 -2.186648937497128
- joint stand_right_arm_base_fixed: origin xyz=0.16285534 -0.18646447 0.56285534 rpy=2.1859138555489475 -0.5231322390070723 -0.9549437348744108 -> xyz=0.16098534 -0.18516447 0.56214534 rpy=2.1859138555489475 -0.5231322390070723 -0.9549437348744108

Commit message: self-collision: 40-hull stand, arm<->stand its own class at 20/62, jaw-tracking highlight
Five related changes to the mesh self-collision model, all measured.

STAND GEOMETRY 20 -> 40 CoACD hulls (threshold 0.08 -> 0.03). The hulls
over-approximate the stand, so the guard reports the arm closer than it is --
padding stacked on d_hard_m, safe but paid out of usable workspace. New tool
rb_servo_server/tools/stand_hull_sweep.py measures it the way that matters: the
clearance the real CollisionMonitor reports at 1500 random arm poses in the
10..150 mm band, against a reference model built from the source STL as a coal
BVH (exact distance). 20 hulls: mean 0.11 / p95 0.03 / MAX 10.82 mm. 40 hulls:
mean 0.05 / p95 0.09 / MAX 5.97 mm. Neither under-approximates (err_min
-0.03 mm = GJK/BVH tolerance). 40 is the finest set whose per-eval p99 stays
under the 2 ms servo tick, i.e. the finest that still gives the async monitor a
verdict PER TICK -- past that it evaluates every other tick, which doubles the
interval swept_samples covers. Shipped STLs are the ones measured, not a
re-run; coacd 1.0.14 with the recorded parameters reproduces them bit-identically.

ARM<->STAND IS ITS OWN BARRIER CLASS, split out of the self set, and tightened
to 20/62 mm (arm<->arm stays 30/75). The two are not the same problem: an
arm<->arm clearance spans two mount calibrations and two DH chains, arm<->stand
carries one arm's error against a structure the same 27-contact calibration
fitted directly. This class's worst unsafe-direction term is the left arm's
5.4 mm box DH oracle, which 20 mm covers 3.7x -- defensible only because the
hull refinement above took the geometry's own padding out of the way first.
Measured effect over the same 1500 poses: below floor 17.2% -> 8.5%.
d_slow 0.062 not 0.060 because the invariant needs exactly 0.060, i.e. zero
headroom against any later change to the TCP ceiling or the shared a_brake.

  * 0 = inherit the self value, resolved WHERE USED, not only in the YAML layer.
    The class was carved out of an existing one, so every caller that builds
    CollisionMonitorConfig directly and sets only d_hard_m -- offline tools, the
    tests -- would otherwise have arm<->stand silently drop to a struct default
    and stop enforcing what it used to. A test caught exactly that.
  * self_min_clearance_m still INCLUDES arm<->stand: the InitMotion planner
    gates on it, and narrowing it would drop the class out of that gate.

HIGHLIGHT OVERLAY FOLLOWS THE JAW. update_self_collision_overlay posed the
articulated arm URDF without a gripper percent, so _finger_position_m(None)
parked the prismatic fingers at FULL OPEN forever: a gripper<->gripper highlight
drew jaws 98 mm apart while the real ones were closed on a bolt. Same fix for
the reference ghost, which the overlay replaces per body group.

TELEMETRY. selfcol_arm_stand_min_clearance_m and selfcol_environment_min_
clearance_m in the servo log and the state stream; both classes enforce their
own d_hard_m and neither had a column, so how close the cell comes to the stand
or the riser was not answerable from a run. near_pairs entries carry the
arm_stand flag. evalOnce now fills CollisionVerdict::eval_ms (it was set only on
the monitor thread, so every synchronous caller read 0 as "free").

collision_pose_probe gains --poses (batch, one model build), --unified-urdf,
--swept, --repeat, an arm<->stand column and the class label, and now honours
the config's swept_samples instead of hardcoding 1 -- its contract is "the same
CollisionMonitor the server builds", and swept_samples is what the cost scales
with. --swept 1 is load-bearing for the sweep: the monitor interpolates from the
PREVIOUS evaluated pose, so unrelated batch poses each "sweep" across the cell.
Before that was pinned, a pose whose true clearance is 82.3 mm reported
-103.8 mm and every variant inherited the same fiction.

ctest 59/59, rb_gui 389/389, --check-config OK on both stacks. Verified the
staged tree builds and tests on its own in a scratch worktree. NOT yet run on
hardware: watch selfcol_eval_ms (projected p50 ~1.16 / p99 ~1.77 ms),
selfcol_verdict_age_ms staying under 2 ms, and the new arm<->stand column.

Co-Authored-By: Claude Opus 5 <noreply@anthropic.com>

File: rb_servo_server/descriptions/urdf/dual_rb5_850e_ver3.urdf (robot description, URDF)
Before this commit: robot dual_rb5_850e_ver1, 29 links, 28 joints
Links:
- link stand_collision: geometry collision mesh filename=../meshes/stands/dual_rb5_850e/collision_ver1/stand_hull_00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 scale=0.001 0.001 0.001; collision mesh filename=../meshes/stands/dual_rb5_850e/collision_ver1/stand_hull_00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 scale=0.001 0.001 0.001
