Commit message: Add environment furniture to URDF generation and implement recorded pose IK audit tool
- Extended `make_rb5_850e_urdfs.py` to include environment furniture (work tables and risers) with visual and collision properties.
- Introduced `_environment_elements` function to handle the creation of environment links and their fixed joints.
- Added `recorded_pose_ik_audit.cpp` to analyze recorded Cartesian targets against actual IK results, ensuring compliance with joint position and rate limits.
- Updated `flow_infer_real_policy.sh` to include new parameters for chunk activation mode and TCP target profile.
- Created `replay_chunk_activation.py` to replay recorded inference durations and evaluate scheduling and timing without constructing models or robots.

File: rb_servo_server/descriptions/urdf/dual_rb5_850e_ver3.urdf (robot description, URDF)
Before this commit: robot dual_rb5_850e_ver2, 30 links, 29 joints
Links:
- added link env_stand_riser; collision box size=0.307 0.324 0.295; visual box size=0.307 0.324 0.295
- added link env_work_table; visual box size=0.8 0.8 0.8
- added link env_work_table_2; visual box size=0.8 0.8 0.8
Joints:
- added joint env_stand_riser_fixed: type fixed, parent stand, child env_stand_riser, origin xyz=0 0.0049 -0.1625 rpy=0.0 0.0 0.0
- added joint env_work_table_2_fixed: type fixed, parent stand, child env_work_table_2, origin xyz=1.05 0 -0.71 rpy=0.0 0.0 0.0
- added joint env_work_table_fixed: type fixed, parent stand, child env_work_table, origin xyz=0.25 0 -0.71 rpy=0.0 0.0 0.0

Commit message: Add collision pose probe tool and update configurations
- Introduced `collision_pose_probe` tool to evaluate self-collision models at recorded joint poses and print nearest pairs with witness points.
- Updated `CMakeLists.txt` to include the new executable for `collision_pose_probe`.
- Modified `stack_real.yaml` to adjust minimum joint limits and added a new UDP endpoint for the collision pose probe tool.
- Updated URDF definitions for `dual_rb5_850e_ver3` to reflect changes in the environment stand riser and added a new spacer link.
- Adjusted tests in `test_collision_monitor.cpp` and `test_config_loader.cpp` to account for the new geometry and configuration changes.
- Enhanced `make_rb5_850e_urdfs.py` to support cylinder shapes for environment elements.
- Added `near_pairs_watch.py` for live monitoring of self-collision guard's near pairs during operation.
- Created `read_wrist_intrinsics.py` to read and print wrist camera intrinsics for inference configuration.
- Updated flow inference script to include new environment variables for wrist camera normalization.

File: rb_servo_server/descriptions/urdf/dual_rb5_850e_ver3.urdf (robot description, URDF)
Before this commit: robot dual_rb5_850e_ver1, 28 links, 27 joints
Links:
- added link env_stand_spacer; collision cylinder length=0.015 radius=0.133; visual cylinder length=0.015 radius=0.133
- link env_stand_riser: geometry collision box size=0.307 0.324 0.28; visual box size=0.307 0.324 0.28
Joints:
- added joint env_stand_spacer_fixed: type fixed, parent stand, child env_stand_spacer, origin xyz=0 0.0049 -0.0225 rpy=0.0 0.0 0.0
- joint env_stand_riser_fixed: origin xyz=0 0.0049 -0.1625 rpy=0.0 0.0 0.0 -> xyz=0 0.0049 -0.17 rpy=0.0 0.0 0.0

Commit message: Add contact-close functionality and update gripper feedback handling
- Implemented ContactCloseConfig and ContactCloseController to manage gripper closing behavior based on motor current feedback.
- Enhanced unit tests for contact-close functionality, ensuring correct state transitions and grip validation.
- Updated rollout step logging to accurately record contact-close verdicts and grip states.
- Adjusted robot configuration files to reflect changes in elbow joint limits, ensuring alignment with mechanical constraints.
- Modified URDF files to maintain consistency with updated elbow bounds and prevent self-collision issues.
- Improved gripper bridge to include contact-close verdicts in feedback messages.
- Enhanced analysis tools to account for new current thresholds during gripping actions.

File: rb_servo_server/descriptions/urdf/dual_rb5_850e_ver3.urdf (robot description, URDF)
Before this commit: robot dual_rb5_850e_ver1, 29 links, 28 joints
Joints:
- joint dual_rb5_850e_left_elbow_joint: limit lower=-2.879793 upper=2.879793 effort=0.0 velocity=3.141592653589793 -> lower=-2.792527 upper=2.792527 effort=0.0 velocity=3.141592653589793
- joint dual_rb5_850e_right_elbow_joint: limit lower=-2.879793 upper=2.879793 effort=0.0 velocity=3.141592653589793 -> lower=-2.792527 upper=2.792527 effort=0.0 velocity=3.141592653589793

File: rb_servo_server/descriptions/urdf/rb5_850e.urdf (robot description, URDF)
Before this commit: robot rb5_850e, 13 links, 12 joints
Joints:
- joint elbow_joint: limit lower=-2.879793 upper=2.879793 effort=0.0 velocity=3.141592653589793 -> lower=-2.792527 upper=2.792527 effort=0.0 velocity=3.141592653589793

File: rb_servo_server/descriptions/urdf/rb5_850e_pika_articulated.urdf (robot description, URDF)
Before this commit: robot rb5_850e, 15 links, 14 joints
Joints:
- joint elbow_joint: limit lower=-2.879793 upper=2.879793 effort=0.0 velocity=3.141592653589793 -> lower=-2.792527 upper=2.792527 effort=0.0 velocity=3.141592653589793
